Commit message: update URDF adding limits to joints

File: CAD_files/URDF/BOTZO_URDF_description/urdf/BOTZO_URDF.urdf (robot description, URDF)
Before this commit: robot BOTZO_URDF, 42 links, 41 joints
Joints:
- joint LF_HAA: limit (none) -> lower=-1.5708 upper=1.5708 effort=500 velocity=10; type continuous -> revolute
- joint LF_HFE: limit (none) -> lower=-1.5708 upper=1.5708 effort=500 velocity=10; type continuous -> revolute
- joint LF_KFE: limit (none) -> lower=-1.5708 upper=1.5708 effort=500 velocity=10; type continuous -> revolute
- joint LF_shank_fixed_LF_FOOT: limit (none) -> lower=0 upper=0 effort=500 velocity=0; type continuous -> revolute
- joint LH_HAA: limit (none) -> lower=-1.5708 upper=1.5708 effort=500 velocity=10; type continuous -> revolute
- joint LH_HFE: limit (none) -> lower=-1.5708 upper=1.5708 effort=500 velocity=10; type continuous -> revolute
- joint LH_KFE: limit (none) -> lower=-1.5708 upper=1.5708 effort=500 velocity=10; type continuous -> revolute
- joint LH_shank_fixed_LH_FOOT: limit (none) -> lower=0 upper=0 effort=500 velocity=0; type continuous -> revolute
- joint RF_HAA: limit (none) -> lower=-1.5708 upper=1.5708 effort=500 velocity=10; type continuous -> revolute
- joint RF_HFE: limit (none) -> lower=-1.5708 upper=1.5708 effort=500 velocity=10; type continuous -> revolute
- joint RF_KFE: limit (none) -> lower=-1.5708 upper=1.5708 effort=500 velocity=10; type continuous -> revolute
- joint RF_shank_fixed_RF_FOOT: limit (none) -> lower=0 upper=0 effort=500 velocity=0; type continuous -> revolute
- joint RH_HAA: limit (none) -> lower=-1.5708 upper=1.5708 effort=500 velocity=10; type continuous -> revolute
- joint RH_HFE: limit (none) -> lower=-1.5708 upper=1.5708 effort=500 velocity=10; type continuous -> revolute
- joint RH_KFE: limit (none) -> lower=-1.5708 upper=1.5708 effort=500 velocity=10; type continuous -> revolute
- joint RH_shank_fixed_RH_FOOT: limit (none) -> lower=0 upper=0 effort=500 velocity=0; type continuous -> revolute

Commit message: new USD tests for RL

File: CAD_files/URDF/BOTZO_URDF_description/urdf/BOTZO_URDF.urdf (robot description, URDF)
Before this commit: robot BOTZO_URDF, 42 links, 41 joints
Links:
- link BL_femur_servo: mass 0.2617 -> 0.2617400479417799
- link BL_hip_holder: mass 0.2738 -> 0.27383943853852916
- link BL_hip_servo: mass 0.2617 -> 0.2617400478829367
- link BL_tibia_servo: mass 0.2617 -> 0.26173858999953525
- link BR_femur_servo: mass 0.2617 -> 0.26174004794177985
- link BR_hip_holder: mass 0.2738 -> 0.2738404315973338
- link BR_hip_servo: mass 0.2617 -> 0.2617400478829346
- link BR_tibia_servo: mass 0.2617 -> 0.2617385899995351
- link FL_femur_servo: mass 0.2617 -> 0.2617400479417799
- link FL_hip_holder: mass 0.2738 -> 0.2739065316373336
- link FL_hip_servo: mass 0.2617 -> 0.26173993659313904
- link FL_tibia_servo: mass 0.2617 -> 0.261739222329772
- link FR_femur_servo: mass 0.2617 -> 0.26174004794177985
- link FR_hip_holder: mass 0.2738 -> 0.2739065893365788
- link FR_hip_servo: mass 0.2617 -> 0.26174004794177985
- link FR_tibia_servo: mass 0.2617 -> 0.2617392223297719
- link LF_FOOT: mass 0.0343 -> 0.034348407017534784
- link LF_HIP: mass 0.0095 -> 0.009507835913863746
- link LF_SHANK: mass 0.164 -> 0.16449852643699206
- link LF_THIGH: mass 0.1232 -> 0.12321527244392107
- link LH_FOOT: mass 0.0343 -> 0.034348407017534784
- link LH_HIP: mass 0.0095 -> 0.009507508379080121
- link LH_SHANK: mass 0.164 -> 0.164498526436992
- link LH_THIGH: mass 0.1232 -> 0.12321527244393736
- link RF_FOOT: mass 0.0343 -> 0.03434778325699268
- link RF_HIP: mass 0.0095 -> 0.009507493907444358
- link RF_SHANK: mass 0.164 -> 0.16449882147273556
- link RF_THIGH: mass 0.1232 -> 0.1232160348472257
- link RH_FOOT: mass 0.0343 -> 0.03434778325699268
- link RH_HIP: mass 0.0095 -> 0.009507457536661807
- link RH_SHANK: mass 0.164 -> 0.16449882147273576
- link RH_THIGH: mass 0.1232 -> 0.1232160348472388
- link face: mass 0.42 -> 0.42237332709158726
- link internal_infra: mass 0.296 -> 0.29688366953182493
- link plaque_left: mass 0.265 -> 0.2650412288141514
- link plaque_right: mass 0.265 -> 0.2662946576400111
- link rear: mass 0.42 -> 0.4112027073712677
- link top: mass 1.115 -> 1.1154165815498167
Joints:
- removed joint LF_shank_fixed_LF_FOOT
- removed joint LH_shank_fixed_LH_FOOT
- removed joint RF_shank_fixed_RF_FOOT
- removed joint RH_shank_fixed_RH_FOOT
- added joint LF_FOOT_link: type fixed, parent LF_SHANK, child LF_FOOT, origin xyz=-0.001225 -0.006586 -0.089906 rpy=0 0 0
- added joint LH_FOOT_link: type fixed, parent LH_SHANK, child LH_FOOT, origin xyz=-0.001225 -0.006586 -0.089906 rpy=0 0 0
- added joint RF_FOOT_link: type fixed, parent RF_SHANK, child RF_FOOT, origin xyz=-0.001225 0.006586 -0.089906 rpy=0 0 0
- added joint RH_FOOT_link: type fixed, parent RH_SHANK, child RH_FOOT, origin xyz=-0.001225 0.006586 -0.089906 rpy=0 0 0

File: CAD_files/URDF/BOTZO_URDF_description/urdf/BOTZO_URDF.xacro (robot description, xacro)
@@ -67,5 +67,5 @@
   <inertial>
     <origin xyz="-0.010978826420354432 0.024635560993822213 0.004999993099930565" rpy="0 0 0"/>
-    <mass value="0.2617"/>
+    <mass value="0.26173993659313904"/>
     <inertia ixx="4.6e-05" iyy="4.4e-05" izz="7.2e-05" ixy="0.0" iyz="-0.0" ixz="-0.0"/>
   </inertial>
@@ -75,5 +75,5 @@
       <mesh filename="../meshes/FL_hip_servo.stl" scale="0.001 0.001 0.001"/>
     </geometry>
-    <material name="shoulder_material"/>
+    <material name="body_material"/>
   </visual>
   <collision>
@@ -87,5 +87,5 @@
   <inertial>
     <origin xyz="0.010978566432420041 0.024635553472565068 0.004999993096986129" rpy="0 0 0"/>
-    <mass value="0.2617"/>
+    <mass value="0.2617400478829367"/>
     <inertia ixx="4.6e-05" iyy="4.4e-05" izz="7.2e-05" ixy="-0.0" iyz="-0.0" ixz="-0.0"/>
   </inertial>
@@ -95,5 +95,5 @@
       <mesh filename="../meshes/BL_hip_servo.stl" scale="0.001 0.001 0.001"/>
     </geometry>
-    <material name="shoulder_material"/>
+    <material name="body_material"/>
   </visual>
   <collision>
@@ -107,5 +107,5 @@
   <inertial>
     <origin xyz="0.010978566432483449 -0.02463554393590102 0.005000000088002207" rpy="0 0 0"/>
-    <mass value="0.2617"/>
+    <mass value="0.2617400478829346"/>
     <inertia ixx="4.6e-05" iyy="4.4e-05" izz="7.2e-05" ixy="0.0" iyz="0.0" ixz="-0.0"/>
   </inertial>
@@ -115,5 +115,5 @@
       <mesh filename="../meshes/BR_hip_servo.stl" scale="0.001 0.001 0.001"/>
     </geometry>
-    <material name="shoulder_material"/>
+    <material name="body_material"/>
   </visual>
   <collision>
@@ -127,5 +127,5 @@
   <inertial>
     <origin xyz="-0.010978819400829183 -0.02463554393111611 0.005000000090946616" rpy="0 0 0"/>
-    <mass value="0.2617"/>
+    <mass value="0.26174004794177985"/>
     <inertia ixx="4.6e-05" iyy="4.4e-05" izz="7.2e-05" ixy="-0.0" iyz="0.0" ixz="-0.0"/>
   </inertial>
@@ -135,5 +135,5 @@
       <mesh filename="../meshes/FR_hip_servo.stl" scale="0.001 0.001 0.001"/>
     </geometry>
-    <material name="shoulder_material"/>
+    <material name="body_material"/>
   </visual>
   <collision>
@@ -147,5 +147,5 @@
   <inertial>
     <origin xyz="-0.0033823271841275857 1.4796413910361794e-05 0.007872333848179133" rpy="0 0 0"/>
-    <mass value="0.0095"/>
+    <mass value="0.009507508379080121"/>
     <inertia ixx="1e-06" iyy="1e-06" izz="0.0" ixy="-0.0" iyz="-0.0" ixz="0.0"/>
   </inertial>
@@ -167,5 +167,5 @@
   <inertial>
     <origin xyz="-0.0033823296605766523 -1.480449380279747e-05 0.00787237940155594" rpy="0 0 0"/>
-    <mass value="0.0095"/>
+    <mass value="0.009507457536661807"/>
     <inertia ixx="1e-06" iyy="1e-06" izz="0.0" ixy="0.0" iyz="0.0" ixz="0.0"/>
   </inertial>
@@ -187,5 +187,5 @@
   <inertial>
     <origin xyz="0.003382077615074093 1.4787446472486199e-05 0.007872350264379872" rpy="0 0 0"/>
-    <mass value="0.0095"/>
+    <mass value="0.009507493907444358"/>
     <inertia ixx="1e-06" iyy="1e-06" izz="0.0" ixy="0.0" iyz="-0.0" ixz="-0.0"/>
   </inertial>
@@ -207,5 +207,5 @@
   <inertial>
     <origin xyz="0.0033820809457219755 -1.45680062756115e-05 0.007871874279300785" rpy="0 0 0"/>
-    <mass value="0.0095"/>
+    <mass value="0.009507835913863746"/>
     <inertia ixx="1e-06" iyy="1e-06" izz="0.0" ixy="-0.0" iyz="0.0" ixz="-0.0"/>
   </inertial>
@@ -227,5 +227,5 @@
   <inertial>
     <origin xyz="0.029560698455582325 -0.0006139250348962816 -0.005293910274418584" rpy="0 0 0"/>
-    <mass value="0.2738"/>
+    <mass value="0.2739065893365788"/>
     <inertia ixx="8.1e-05" iyy="0.000224" izz="0.000184" ixy="1e-06" iyz="-1e-06" ixz="-1.2e-05"/>
   </inertial>
@@ -247,5 +247,5 @@
   <inertial>
     <origin xyz="0.029560702894754244 0.0006139344660216831 -0.005293914635593616" rpy="0 0 0"/>
-    <mass value="0.2738"/>
+    <mass value="0.2739065316373336"/>
     <inertia ixx="8.1e-05" iyy="0.000224" izz="0.000184" ixy="-1e-06" iyz="1e-06" ixz="-1.2e-05"/>
   </inertial>
@@ -267,5 +267,5 @@
   <inertial>
     <origin xyz="-0.029567418713488176 -0.0006140698430923894 -0.005290300978496018" rpy="0 0 0"/>
-    <mass value="0.2738"/>
+    <mass value="0.2738404315973338"/>
     <inertia ixx="8.1e-05" iyy="0.000224" izz="0.000184" ixy="-1e-06" iyz="-1e-06" ixz="1.2e-05"/>
   </inertial>
@@ -287,5 +287,5 @@
   <inertial>
     <origin xyz="-0.02956749620152093 0.0006140814047106841 -0.005290344095366009" rpy="0 0 0"/>
-    <mass value="0.2738"/>
+    <mass value="0.27383943853852916"/>
     <inertia ixx="8.1e-05" iyy="0.000224" izz="0.000184" ixy="1e-06" iyz="1e-06" ixz="1.2e-05"/>
   </inertial>
@@ -307,5 +307,5 @@
   <inertial>
     <origin xyz="-0.024964370616050904 0.010978365390125422 0.004999649993067221" rpy="0 0 0"/>
-    <mass value="0.2617"/>
+    <mass value="0.2617400479417799"/>
     <inertia ixx="4.4e-05" iyy="4.6e-05" izz="7.2e-05" ixy="-0.0" iyz="0.0" ixz="-0.0"/>
   </inertial>
@@ -327,5 +327,5 @@
   <inertial>
     <origin xyz="-0.02463534146393219 0.010978408940392835 0.0049996411984006145" rpy="0 0 0"/>
-    <mass value="0.2617"/>
+    <mass value="0.26173858999953525"/>
     <inertia ixx="4.4e-05" iyy="4.6e-05" izz="7.2e-05" ixy="0.0" iyz="-0.0" ixz="-0.0"/>
   </inertial>
@@ -347,5 +347,5 @@
   <inertial>
     <origin xyz="-0.024964370616009382 -0.010978355853619524 0.004999656984075548" rpy="0 0 0"/>
-    <mass value="0.2617"/>
+    <mass value="0.26174004794177985"/>
     <inertia ixx="4.4e-05" iyy="4.6e-05" izz="7.2e-05" ixy="0.0" iyz="-0.0" ixz="-0.0"/>
   </inertial>
@@ -367,5 +367,5 @@
   <inertial>
     <origin xyz="-0.0246353414638866 -0.010978399403886119 0.004999648189409005" rpy="0 0 0"/>
-    <mass value="0.2617"/>
+    <mass value="0.2617385899995351"/>
     <inertia ixx="4.4e-05" iyy="4.6e-05" izz="7.2e-05" ixy="-0.0" iyz="0.0" ixz="-0.0"/>
   </inertial>
@@ -387,5 +387,5 @@
   <inertial>
     <origin xyz="0.024635236782420036 0.010978365390344982 0.004999645985760567" rpy="0 0 0"/>
-    <mass value="0.2617"/>
+    <mass value="0.2617400479417799"/>
     <inertia ixx="4.4e-05" iyy="4.6e-05" izz="7.2e-05" ixy="-0.0" iyz="0.0" ixz="-0.0"/>
   </inertial>
@@ -407,5 +407,5 @@
   <inertial>
     <origin xyz="0.024964033753852463 0.010978390052187453 0.004999641006598471" rpy="0 0 0"/>
-    <mass value="0.2617"/>
+    <mass value="0.261739222329772"/>
     <inertia ixx="4.4e-05" iyy="4.6e-05" izz="7.2e-05" ixy="0.0" iyz="-0.0" ixz="0.0"/>
   </inertial>
@@ -427,5 +427,5 @@
   <inertial>
     <origin xyz="0.02463523678246525 -0.010978355853581062 0.004999652976776514" rpy="0 0 0"/>
-    <mass value="0.2617"/>
+    <mass value="0.26174004794177985"/>
     <inertia ixx="4.4e-05" iyy="4.6e-05" izz="7.2e-05" ixy="0.0" iyz="-0.0" ixz="-0.0"/>
   </inertial>
@@ -447,5 +447,5 @@
   <inertial>
     <origin xyz="0.024964033753897955 -0.010978380515422506 0.004999647997614584" rpy="0 0 0"/>
-    <mass value="0.2617"/>
+    <mass value="0.2617392223297719"/>
     <inertia ixx="4.4e-05" iyy="4.6e-05" izz="7.2e-05" ixy="-0.0" iyz="0.0" ixz="0.0"/>
   </inertial>
@@ -487,5 +487,5 @@
   <inertial>
     <origin xyz="-0.0015487128805810324 0.00818635524879402 -0.046699032368199875" rpy="0 0 0"/>
-    <mass value="0.1232"/>
+    <mass value="0.12321527244392107"/>
     <inertia ixx="0.000112" iyy="0.000111" izz="6e-06" ixy="-0.0" iyz="-2e-06" ixz="-4e-06"/>
   </inertial>
@@ -507,5 +507,5 @@
   <inertial>
     <origin xyz="-0.001548689561858288 -0.00818632723111587 -0.04669919641913074" rpy="0 0 0"/>
-    <mass value="0.1232"/>
+    <mass value="0.1232160348472257"/>
     <inertia ixx="0.000112" iyy="0.000111" izz="6e-06" ixy="0.0" iyz="2e-06" ixz="-4e-06"/>
   </inertial>
@@ -527,5 +527,5 @@
   <inertial>
     <origin xyz="-0.0015481950136371492 -0.008186327231335055 -0.046697922551068013" rpy="0 0 0"/>
-    <mass value="0.1232"/>
+    <mass value="0.1232160348472388"/>
     <inertia ixx="0.000112" iyy="0.000111" izz="6e-06" ixy="0.0" iyz="2e-06" ixz="-4e-06"/>
   </inertial>
@@ -546,6 +546,6 @@
 <link name="LH_THIGH">
   <inertial>
-    <origin xyz="-0.0015481437644143808 0.008186355248752455 -0.0466975963630347" rpy="0 0 0"/>
-    <mass value="0.1232"/>
+    <origin xyz="-0.0015481437644144225 0.008186355248752455 -0.0466975963630347" rpy="0 0 0"/>
+    <mass value="0.12321527244393736"/>
     <inertia ixx="0.000113" iyy="0.000111" izz="6e-06" ixy="-0.0" iyz="-2e-06" ixz="-4e-06"/>
   </inertial>
@@ -564,9 +564,169 @@
   </collision>
 </link>
+<link name="plaque_left">
+  <inertial>
+    <origin xyz="0.014393569624221867 -0.02888533887184032 0.007166851005990391" rpy="0 0 0"/>
+    <mass value="0.2650412288141514"/>
+    <inertia ixx="0.000113" iyy="0.000207" izz="0.000285" ixy="0.0" iyz="8e-06" ixz="0.0"/>
+  </inertial>
+  <visual>
+    <origin xyz="0.00664 0.018475 -0.0624" rpy="0 0 0"/>
+    <geometry>
+      <mesh filename="../meshes/plaque_left.stl" scale="0.001 0.001 0.001"/>
+    </geometry>
+    <material name="body_material"/>
+  </visual>
+  <collision>
+    <origin xyz="0.00664 0.018475 -0.0624" rpy="0 0 0"/>
+    <geometry>
+      <mesh filename="../meshes/plaque_left.stl" scale="0.001 0.001 0.001"/>
+    </geometry>
+  </collision>
+</link>
+<link name="plaque_right">
+  <inertial>
+    <origin xyz="0.01437999212800966 0.028910459753787983 0.007144962390201057" rpy="0 0 0"/>
+    <mass value="0.2662946576400111"/>
+    <inertia ixx="0.000113" iyy="0.000208" izz="0.000286" ixy="-0.0" iyz="-8e-06" ixz="-0.0"/>
+  </inertial>
+  <visual>
+    <origin xyz="0.00664 -0.018475 -0.0624" rpy="0 0 0"/>
+    <geometry>
+      <mesh filename="../meshes/plaque_right.stl" scale="0.001 0.001 0.001"/>
+    </geometry>
+    <material name="body_material"/>
+  </visual>
+  <collision>
+    <origin xyz="0.00664 -0.018475 -0.0624" rpy="0 0 0"/>
+    <geometry>
+      <mesh filename="../meshes/plaque_right.stl" scale="0.001 0.001 0.001"/>
+    </geometry>
+  </collision>
+</link>
+<link name="rear">
+  <inertial>
+    <origin xyz="-0.002467088490467728 0.01679061879749418 0.03991220570023193" rpy="0 0 0"/>
+    <mass value="0.4112027073712677"/>
+    <inertia ixx="0.000826" iyy="0.000229" izz="0.000599" ixy="0.0" iyz="1.1e-05" ixz="0.0"/>
+  </inertial>
+  <visual>
+    <origin xyz="0.107742 0.015621 -0.0385" rpy="0 0 0"/>
+    <geometry>
+      <mesh filename="../meshes/rear.stl" scale="0.001 0.001 0.001"/>
+    </geometry>
+    <material name="body_material"/>
+  </visual>
+  <collision>
+    <origin xyz="0.107742 0.015621 -0.0385" rpy="0 0 0"/>
+    <geometry>
+      <mesh filename="../meshes/rear.stl" scale="0.001 0.001 0.001"/>
+    </geometry>
+  </collision>
+</link>
+<link name="face">
+  <inertial>
+    <origin xyz="0.0024414347125266272 0.015621074926330704 0.03876987732727693" rpy="0 0 0"/>
+    <mass value="0.42237332709158726"/>
+    <inertia ixx="0.000844" iyy="0.000239" izz="0.000607" ixy="0.0" iyz="-0.0" ixz="-0.0"/>
+  </inertial>
+  <visual>
+    <origin xyz="-0.123238 0.015621 -0.0385" rpy="0 0 0"/>
+    <geometry>
+      <mesh filename="../meshes/face.stl" scale="0.001 0.001 0.001"/>
+    </geometry>
+    <material name="body_material"/>
+  </visual>
+  <collision>
+    <origin xyz="-0.123238 0.015621 -0.0385" rpy="0 0 0"/>
+    <geometry>
+      <mesh filename="../meshes/face.stl" scale="0.001 0.001 0.001"/>
+    </geometry>
+  </collision>
+</link>
+<link name="internal_infra">
+  <inertial>
+    <origin xyz="0.11530993699758461 0.044680485707850826 -0.007028415436090132" rpy="0 0 0"/>
+    <mass value="0.29688366953182493"/>
+    <inertia ixx="0.000331" iyy="0.001813" izz="0.002141" ixy="0.0" iyz="1e-06" ixz="0.0"/>
+  </inertial>
+  <visual>
+    <origin xyz="0.107742 0.043961 -0.105071" rpy="0 0 0"/>
+    <geometry>
+      <mesh filename="../meshes/internal_infra.stl" scale="0.001 0.001 0.001"/>
+    </geometry>
+    <material name="body_material"/>
+  </visual>
+  <collision>
+    <origin xyz="0.107742 0.043961 -0.105071" rpy="0 0 0"/>
+    <geometry>
+      <mesh filename="../meshes/internal_infra.stl" scale="0.001 0.001 0.001"/>
+    </geometry>
+  </collision>
+</link>
+<link name="top">
+  <inertial>
+    <origin xyz="0.11761953860342345 -0.06398448625003379 0.011181156410446563" rpy="0 0 0"/>
+    <mass value="1.1154165815498167"/>
+    <inertia ixx="0.002509" iyy="0.005671" izz="0.007973" ixy="3.8e-05" iyz="-2.2e-05" ixz="-3e-06"/>
+  </inertial>
+  <visual>
+    <origin xyz="0.110242 -0.0616 -0.105415" rpy="0 0 0"/>
+    <geometry>
+      <mesh filename="../meshes/top.stl" scale="0.001 0.001 0.001"/>
+    </geometry>
+    <material name="body_material"/>
+  </visual>
+  <collision>
+    <origin xyz="0.110242 -0.0616 -0.105415" rpy="0 0 0"/>
+    <geometry>
+      <mesh filename="../meshes/top.stl" scale="0.001 0.001 0.001"/>
+    </geometry>
+  </collision>
+</link>
+<link name="RF_SHANK">
+  <inertial>
+    <origin xyz="-1.3426662960558389e-05 0.006598316213941233 -0.04761054175330333" rpy="0 0 0"/>
+    <mass value="0.16449882147273556"/>
+    <inertia ixx="0.000143" iyy="0.000134" izz="1.5e-05" ixy="-0.0" iyz="0.0" ixz="3e-06"/>
+  </inertial>
+  <visual>
+    <origin xyz="-0.079571 0.0849 0.019458" rpy="0 0 0"/>
+    <geometry>
+      <mesh filename="../meshes/RF_SHANK.stl" scale="0.001 0.001 0.001"/>
+    </geometry>
+    <material name="legs_material"/>
+  </visual>
+  <collision>
+    <origin xyz="-0.079571 0.0849 0.019458" rpy="0 0 0"/>
+    <geometry>
+      <mesh filename="../meshes/RF_SHANK.stl" scale="0.001 0.001 0.001"/>
+    </geometry>
+  </collision>
+</link>
+<link name="RH_SHANK">
+  <inertial>
+    <origin xyz="-1.3034061444691658e-05 0.00659831600262395 -0.04761053774599561" rpy="0 0 0"/>
+    <mass value="0.16449882147273576"/>
+    <inertia ixx="0.000143" iyy="0.000134" izz="1.5e-05" ixy="-0.0" iyz="0.0" ixz="3e-06"/>
+  </inertial>
+  <visual>
+    <origin xyz="0.084076 0.0849 0.019458" rpy="0 0 0"/>
+    <geometry>
+      <mesh filename="../meshes/RH_SHANK.stl" scale="0.001 0.001 0.001"/>
+    </geometry>
+    <material name="legs_material"/>
+  </visual>
+  <collision>
+    <origin xyz="0.084076 0.0849 0.019458" rpy="0 0 0"/>
+    <geometry>
+      <mesh filename="../meshes/RH_SHANK.stl" scale="0.001 0.001 0.001"/>
+    </geometry>
+  </collision>
+</link>
 <link name="LF_SHANK">
   <inertial>
-    <origin xyz="0.04761573643303946 -0.006599694761353192 -1.2592420719485797e-05" rpy="0 0 0"/>
-    <mass value="0.164"/>
-    <inertia ixx="1.5e-05" iyy="0.000134" izz="0.000143" ixy="-0.0" iyz="0.0" ixz="-3e-06"/>
+    <origin xyz="-1.3423486317318267e-05 -0.006598286312571797 -0.047610458897788074" rpy="0 0 0"/>
+    <mass value="0.16449852643699206"/>
+    <inertia ixx="0.000143" iyy="0.000134" izz="1.5e-05" ixy="0.0" iyz="-0.0" ixz="3e-06"/>
   </inertial>
   <visual>
@@ -584,61 +744,61 @@
   </collision>
 </link>
-<link name="RF_SHANK">
-  <inertial>
-    <origin xyz="0.04761036870481894 0.006598316213817332 -1.353852544248857e-05" rpy="0 0 0"/>
-    <mass value="0.164"/>
-    <inertia ixx="1.5e-05" iyy="0.000134" izz="0.000143" ixy="-0.0" iyz="-0.0" ixz="-3e-06"/>
-  </inertial>
-  <visual>
-    <origin xyz="-0.079571 0.0849 0.019458" rpy="0 0 0"/>
-    <geometry>
-      <mesh filename="../meshes/RF_SHANK.stl" scale="0.001 0.001 0.001"/>
+<link name="LH_SHANK">
+  <inertial>
+    <origin xyz="-1.3030884784909214e-05 -0.006598286101516498 -0.0476104548904905" rpy="0 0 0"/>
+    <mass value="0.164498526436992"/>
+    <inertia ixx="0.000143" iyy="0.000134" izz="1.5e-05" ixy="0.0" iyz="-0.0" ixz="3e-06"/>
+  </inertial>
+  <visual>
+    <origin xyz="0.084076 -0.0849 0.019458" rpy="0 0 0"/>
+    <geometry>
+      <mesh filename="../meshes/LH_SHANK.stl" scale="0.001 0.001 0.001"/>
     </geometry>
     <material name="legs_material"/>
   </visual>
   <collision>
-    <origin xyz="-0.079571 0.0849 0.019458" rpy="0 0 0"/>
-    <geometry>
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