Commit message: new urdf with new materials

File: botzo_ros2_ws/urdf/botzo.urdf (robot description, URDF)
Before this commit: robot BOTZO_URDF, 42 links, 41 joints
Links:
- removed link BL_femur_servo
- removed link BL_hip_holder
- removed link BL_hip_servo
- removed link BL_tibia_servo
- removed link BR_femur_servo
- removed link BR_hip_holder
- removed link BR_hip_servo
- removed link BR_tibia_servo
- removed link FL_femur_servo
- removed link FL_hip_holder
- removed link FL_hip_servo
- removed link FL_tibia_servo
- removed link FR_femur_servo
- removed link FR_hip_holder
- removed link FR_hip_servo
- removed link FR_tibia_servo
- removed link LF_FOOT
- removed link LF_HIP
- removed link LF_SHANK
- removed link LF_THIGH
- removed link LH_FOOT
- removed link LH_HIP
- removed link LH_SHANK
- removed link LH_THIGH
- removed link RF_FOOT
- removed link RF_HIP
- removed link RF_SHANK
- removed link RF_THIGH
- removed link RH_FOOT
- removed link RH_HIP
- removed link RH_SHANK
- removed link RH_THIGH
- removed link battery_case
- removed link battery_lid
- removed link face
- removed link imu_link
- removed link internal_infra
- removed link plaque_left
- removed link plaque_right
- removed link rear
- removed link top
- added link BL_femur, mass 0.016638088782005175; collision mesh filename=package://botzo_ros2_ws/urdf/meshes/BL_femur.stl scale=0.001 0.001 0.001; visual mesh filename=package://botzo_ros2_ws/urdf/meshes/BL_femur.stl scale=0.001 0.001 0.001
- added link BL_shoulder, mass 0.10894741172095637; collision mesh filename=package://botzo_ros2_ws/urdf/meshes/BL_shoulder.stl scale=0.001 0.001 0.001; visual mesh filename=package://botzo_ros2_ws/urdf/meshes/BL_shoulder.stl scale=0.001 0.001 0.001
- added link BL_tibia, mass 0.026850714584678158; collision mesh filename=package://botzo_ros2_ws/urdf/meshes/BL_tibia.stl scale=0.001 0.001 0.001; visual mesh filename=package://botzo_ros2_ws/urdf/meshes/BL_tibia.stl scale=0.001 0.001 0.001
- added link BR_femur, mass 0.0166380470560182; collision mesh filename=package://botzo_ros2_ws/urdf/meshes/BR_femur.stl scale=0.001 0.001 0.001; visual mesh filename=package://botzo_ros2_ws/urdf/meshes/BR_femur.stl scale=0.001 0.001 0.001
- added link BR_shoulder, mass 0.10894732734955483; collision mesh filename=package://botzo_ros2_ws/urdf/meshes/BR_shoulder.stl scale=0.001 0.001 0.001; visual mesh filename=package://botzo_ros2_ws/urdf/meshes/BR_shoulder.stl scale=0.001 0.001 0.001
- added link BR_tibia, mass 0.0268506747454801; collision mesh filename=package://botzo_ros2_ws/urdf/meshes/BR_tibia.stl scale=0.001 0.001 0.001; visual mesh filename=package://botzo_ros2_ws/urdf/meshes/BR_tibia.stl scale=0.001 0.001 0.001
- added link FL_femur, mass 0.01663808878200678; collision mesh filename=package://botzo_ros2_ws/urdf/meshes/FL_femur.stl scale=0.001 0.001 0.001; visual mesh filename=package://botzo_ros2_ws/urdf/meshes/FL_femur.stl scale=0.001 0.001 0.001
- added link FL_shoulder, mass 0.10895629411716044; collision mesh filename=package://botzo_ros2_ws/urdf/meshes/FL_shoulder.stl scale=0.001 0.001 0.001; visual mesh filename=package://botzo_ros2_ws/urdf/meshes/FL_shoulder.stl scale=0.001 0.001 0.001
- added link FL_tibia, mass 0.026850714584678873; collision mesh filename=package://botzo_ros2_ws/urdf/meshes/FL_tibia.stl scale=0.001 0.001 0.001; visual mesh filename=package://botzo_ros2_ws/urdf/meshes/FL_tibia.stl scale=0.001 0.001 0.001
- added link FR_femur, mass 0.01663804705601809; collision mesh filename=package://botzo_ros2_ws/urdf/meshes/FR_femur.stl scale=0.001 0.001 0.001; visual mesh filename=package://botzo_ros2_ws/urdf/meshes/FR_femur.stl scale=0.001 0.001 0.001
- added link FR_shoulder, mass 0.1089563019083912; collision mesh filename=package://botzo_ros2_ws/urdf/meshes/FR_shoulder.stl scale=0.001 0.001 0.001; visual mesh filename=package://botzo_ros2_ws/urdf/meshes/FR_shoulder.stl scale=0.001 0.001 0.001
- added link FR_tibia, mass 0.02685067474548009; collision mesh filename=package://botzo_ros2_ws/urdf/meshes/FR_tibia.stl scale=0.001 0.001 0.001; visual mesh filename=package://botzo_ros2_ws/urdf/meshes/FR_tibia.stl scale=0.001 0.001 0.001
- link base: mass 1.2167441545851616 -> 0.7893620452930467
Joints:
- removed joint LF_HAA
- removed joint LF_HFE
- removed joint LF_KFE
- removed joint LF_shank_fixed_LF_FOOT
- removed joint LH_HAA
- removed joint LH_HFE
- removed joint LH_KFE
- removed joint LH_shank_fixed_LH_FOOT
- removed joint RF_HAA
- removed joint RF_HFE
- removed joint RF_KFE
- removed joint RF_shank_fixed_RF_FOOT
- removed joint RH_HAA
- removed joint RH_HFE
- removed joint RH_KFE
- removed joint RH_shank_fixed_RH_FOOT
- removed joint Rigid 1
- removed joint Rigid 11
- removed joint Rigid 12
- removed joint Rigid 13
- removed joint Rigid 14
- removed joint Rigid 15
- removed joint Rigid 16
- removed joint Rigid 17
- removed joint Rigid 18
- removed joint Rigid 19
- removed joint Rigid 2
- removed joint Rigid 20
- removed joint Rigid 21
- removed joint Rigid 22
- removed joint Rigid 3
- removed joint Rigid 36
- removed joint Rigid 37
- removed joint Rigid 38
- removed joint Rigid 39
- removed joint Rigid 4
- removed joint Rigid 40
- removed joint Rigid 41
- removed joint Rigid 5
- removed joint Rigid 6
- removed joint imu_joint
- added joint Revolute 1: type continuous, parent base, child BL_shoulder, origin xyz=-0.04255 -0.0531 0.0522 rpy=0 0 0, axis -1.0 -0.0 -0.0
- added joint Revolute 10: type continuous, parent BR_femur, child BR_tibia, origin xyz=-0.090579 0.013 4e-06 rpy=0 0 0, axis -0.0 1.0 0.000241
- added joint Revolute 11: type continuous, parent BL_shoulder, child BL_femur, origin xyz=-0.029173 -0.018799 -0.001585 rpy=0 0 0, axis -0.0 1.0 0.000326
- added joint Revolute 12: type continuous, parent BL_femur, child BL_tibia, origin xyz=-0.090579 -0.013 -4e-06 rpy=0 0 0, axis -0.0 1.0 0.000326
- added joint Revolute 2: type continuous, parent base, child BR_shoulder, origin xyz=-0.04255 0.0531 0.0522 rpy=0 0 0, axis 1.0 0.0 0.0
- added joint Revolute 3: type continuous, parent base, child FL_shoulder, origin xyz=0.04255 -0.0531 0.0522 rpy=0 0 0, axis -1.0 -0.0 0.0
- added joint Revolute 4: type continuous, parent base, child FR_shoulder, origin xyz=0.04255 0.0531 0.0522 rpy=0 0 0, axis 1.0 -0.0 -0.0
- added joint Revolute 5: type continuous, parent FR_shoulder, child FR_femur, origin xyz=0.048573 0.0188 -0.001579 rpy=0 0 0, axis 0.0 1.0 0.0
- added joint Revolute 6: type continuous, parent FR_femur, child FR_tibia, origin xyz=-0.090579 0.013 0.0 rpy=0 0 0, axis 0.0 1.0 0.0
- added joint Revolute 7: type continuous, parent FL_shoulder, child FL_femur, origin xyz=0.048573 -0.0188 -0.001575 rpy=0 0 0, axis -0.0 1.0 -0.000213
- added joint Revolute 8: type continuous, parent FL_femur, child FL_tibia, origin xyz=-0.090579 -0.013 3e-06 rpy=0 0 0, axis -0.0 1.0 -0.000213
- added joint Revolute 9: type continuous, parent BR_shoulder, child BR_femur, origin xyz=-0.029173 0.018801 -0.001575 rpy=0 0 0, axis -0.0 1.0 0.000241

Commit message: change joints names

File: botzo_ros2_ws/urdf/botzo.urdf (robot description, URDF)
Before this commit: robot botzo, 13 links, 12 joints
Joints:
- removed joint Revolute 1
- removed joint Revolute 10
- removed joint Revolute 11
- removed joint Revolute 12
- removed joint Revolute 2
- removed joint Revolute 3
- removed joint Revolute 4
- removed joint Revolute 5
- removed joint Revolute 6
- removed joint Revolute 7
- removed joint Revolute 8
- removed joint Revolute 9
- added joint BL_femur_joint: type continuous, parent BL_shoulder, child BL_femur, origin xyz=-0.029173 -0.018799 -0.001585 rpy=0 0 0, axis -0.0 1.0 0.000326
- added joint BL_shoulder_joint: type continuous, parent base, child BL_shoulder, origin xyz=-0.04255 -0.0531 0.0522 rpy=0 0 0, axis -1.0 -0.0 -0.0
- added joint BL_tibia_joint: type continuous, parent BL_femur, child BL_tibia, origin xyz=-0.090579 -0.013 -4e-06 rpy=0 0 0, axis -0.0 1.0 0.000326
- added joint BR_femur_joint: type continuous, parent BR_shoulder, child BR_femur, origin xyz=-0.029173 0.018801 -0.001575 rpy=0 0 0, axis -0.0 1.0 0.000241
- added joint BR_shoulder_joint: type continuous, parent base, child BR_shoulder, origin xyz=-0.04255 0.0531 0.0522 rpy=0 0 0, axis 1.0 0.0 0.0
- added joint BR_tibia_joint: type continuous, parent BR_femur, child BR_tibia, origin xyz=-0.090579 0.013 4e-06 rpy=0 0 0, axis -0.0 1.0 0.000241
- added joint FL_femur_joint: type continuous, parent FL_shoulder, child FL_femur, origin xyz=0.048573 -0.0188 -0.001575 rpy=0 0 0, axis -0.0 1.0 -0.000213
- added joint FL_shoulder_joint: type continuous, parent base, child FL_shoulder, origin xyz=0.04255 -0.0531 0.0522 rpy=0 0 0, axis -1.0 -0.0 0.0
- added joint FL_tibia_joint: type continuous, parent FL_femur, child FL_tibia, origin xyz=-0.090579 -0.013 3e-06 rpy=0 0 0, axis -0.0 1.0 -0.000213
- added joint FR_femur_joint: type continuous, parent FR_shoulder, child FR_femur, origin xyz=0.048573 0.0188 -0.001579 rpy=0 0 0, axis 0.0 1.0 0.0
- added joint FR_shoulder_joint: type continuous, parent base, child FR_shoulder, origin xyz=0.04255 0.0531 0.0522 rpy=0 0 0, axis 1.0 -0.0 -0.0
- added joint FR_tibia_joint: type continuous, parent FR_femur, child FR_tibia, origin xyz=-0.090579 0.013 0.0 rpy=0 0 0, axis 0.0 1.0 0.0
