Commit message: setup botzo_description package

File: botzo_ros2_ws/botzo_description/urdf/botzo.urdf (robot description, URDF)
Before this commit: robot botzo, 13 links, 12 joints
Links:
- link BL_femur: geometry collision mesh filename=package://botzo_description/meshes/BL_femur.stl scale=0.001 0.001 0.001; visual mesh filename=package://botzo_description/meshes/BL_femur.stl scale=0.001 0.001 0.001
- link BL_shoulder: geometry collision mesh filename=package://botzo_description/meshes/BL_shoulder.stl scale=0.001 0.001 0.001; visual mesh filename=package://botzo_description/meshes/BL_shoulder.stl scale=0.001 0.001 0.001
- link BL_tibia: geometry collision mesh filename=package://botzo_description/meshes/BL_tibia.stl scale=0.001 0.001 0.001; visual mesh filename=package://botzo_description/meshes/BL_tibia.stl scale=0.001 0.001 0.001
- link BR_femur: geometry collision mesh filename=package://botzo_description/meshes/BR_femur.stl scale=0.001 0.001 0.001; visual mesh filename=package://botzo_description/meshes/BR_femur.stl scale=0.001 0.001 0.001
- link BR_shoulder: geometry collision mesh filename=package://botzo_description/meshes/BR_shoulder.stl scale=0.001 0.001 0.001; visual mesh filename=package://botzo_description/meshes/BR_shoulder.stl scale=0.001 0.001 0.001
- link BR_tibia: geometry collision mesh filename=package://botzo_description/meshes/BR_tibia.stl scale=0.001 0.001 0.001; visual mesh filename=package://botzo_description/meshes/BR_tibia.stl scale=0.001 0.001 0.001
- link FL_femur: geometry collision mesh filename=package://botzo_description/meshes/FL_femur.stl scale=0.001 0.001 0.001; visual mesh filename=package://botzo_description/meshes/FL_femur.stl scale=0.001 0.001 0.001
- link FL_shoulder: geometry collision mesh filename=package://botzo_description/meshes/FL_shoulder.stl scale=0.001 0.001 0.001; visual mesh filename=package://botzo_description/meshes/FL_shoulder.stl scale=0.001 0.001 0.001
- link FL_tibia: geometry collision mesh filename=package://botzo_description/meshes/FL_tibia.stl scale=0.001 0.001 0.001; visual mesh filename=package://botzo_description/meshes/FL_tibia.stl scale=0.001 0.001 0.001
- link FR_femur: geometry collision mesh filename=package://botzo_description/meshes/FR_femur.stl scale=0.001 0.001 0.001; visual mesh filename=package://botzo_description/meshes/FR_femur.stl scale=0.001 0.001 0.001
- link FR_shoulder: geometry collision mesh filename=package://botzo_description/meshes/FR_shoulder.stl scale=0.001 0.001 0.001; visual mesh filename=package://botzo_description/meshes/FR_shoulder.stl scale=0.001 0.001 0.001
- link FR_tibia: geometry collision mesh filename=package://botzo_description/meshes/FR_tibia.stl scale=0.001 0.001 0.001; visual mesh filename=package://botzo_description/meshes/FR_tibia.stl scale=0.001 0.001 0.001
- link base: geometry collision mesh filename=package://botzo_description/meshes/base.stl scale=0.001 0.001 0.001; visual mesh filename=package://botzo_description/meshes/base.stl scale=0.001 0.001 0.001

Commit message: set up gazebo

File: botzo_ros2_ws/botzo_description/urdf/botzo.urdf (robot description, URDF)
Before this commit: robot botzo, 13 links, 12 joints
Links:
- link BL_femur: geometry collision mesh filename=/home/gringo/ros2_ws/src/botzo/botzo_ros2_ws/botzo_descript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 scale=0.001 0.001 0.001; visual mesh filename=/home/gringo/ros2_ws/src/botzo/botzo_ros2_ws/botzo_descript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 scale=0.001 0.001 0.001
- link BL_shoulder: geometry collision mesh filename=/home/gringo/ros2_ws/src/botzo/botzo_ros2_ws/botzo_descript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 scale=0.001 0.001 0.001; visual mesh filename=/home/gringo/ros2_ws/src/botzo/botzo_ros2_ws/botzo_descript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 scale=0.001 0.001 0.001
- link BL_tibia: geometry collision mesh filename=/home/gringo/ros2_ws/src/botzo/botzo_ros2_ws/botzo_descript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 scale=0.001 0.001 0.001; visual mesh filename=/home/gringo/ros2_ws/src/botzo/botzo_ros2_ws/botzo_descript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 scale=0.001 0.001 0.001
- link BR_femur: geometry collision mesh filename=/home/gringo/ros2_ws/src/botzo/botzo_ros2_ws/botzo_descript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 scale=0.001 0.001 0.001; visual mesh filename=/home/gringo/ros2_ws/src/botzo/botzo_ros2_ws/botzo_descript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 scale=0.001 0.001 0.001
- link BR_shoulder: geometry collision mesh filename=/home/gringo/ros2_ws/src/botzo/botzo_ros2_ws/botzo_descript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 scale=0.001 0.001 0.001; visual mesh filename=/home/gringo/ros2_ws/src/botzo/botzo_ros2_ws/botzo_descript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 scale=0.001 0.001 0.001
- link BR_tibia: geometry collision mesh filename=/home/gringo/ros2_ws/src/botzo/botzo_ros2_ws/botzo_descript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 scale=0.001 0.001 0.001; visual mesh filename=/home/gringo/ros2_ws/src/botzo/botzo_ros2_ws/botzo_descript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 scale=0.001 0.001 0.001
- link FL_femur: geometry collision mesh filename=/home/gringo/ros2_ws/src/botzo/botzo_ros2_ws/botzo_descript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 scale=0.001 0.001 0.001; visual mesh filename=/home/gringo/ros2_ws/src/botzo/botzo_ros2_ws/botzo_descript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 scale=0.001 0.001 0.001
- link FL_shoulder: geometry collision mesh filename=/home/gringo/ros2_ws/src/botzo/botzo_ros2_ws/botzo_descript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 scale=0.001 0.001 0.001; visual mesh filename=/home/gringo/ros2_ws/src/botzo/botzo_ros2_ws/botzo_descript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 scale=0.001 0.001 0.001
- link FL_tibia: geometry collision mesh filename=/home/gringo/ros2_ws/src/botzo/botzo_ros2_ws/botzo_descript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 scale=0.001 0.001 0.001; visual mesh filename=/home/gringo/ros2_ws/src/botzo/botzo_ros2_ws/botzo_descript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 scale=0.001 0.001 0.001
- link FR_femur: geometry collision mesh filename=/home/gringo/ros2_ws/src/botzo/botzo_ros2_ws/botzo_descript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 scale=0.001 0.001 0.001; visual mesh filename=/home/gringo/ros2_ws/src/botzo/botzo_ros2_ws/botzo_descript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 scale=0.001 0.001 0.001
- link FR_shoulder: geometry collision mesh filename=/home/gringo/ros2_ws/src/botzo/botzo_ros2_ws/botzo_descript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 scale=0.001 0.001 0.001; visual mesh filename=/home/gringo/ros2_ws/src/botzo/botzo_ros2_ws/botzo_descript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 scale=0.001 0.001 0.001
- link FR_tibia: geometry collision mesh filename=/home/gringo/ros2_ws/src/botzo/botzo_ros2_ws/botzo_descript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 scale=0.001 0.001 0.001; visual mesh filename=/home/gringo/ros2_ws/src/botzo/botzo_ros2_ws/botzo_descript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 scale=0.001 0.001 0.001
- link base: geometry collision mesh filename=/home/gringo/ros2_ws/src/botzo/botzo_ros2_ws/botzo_descript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 scale=0.001 0.001 0.001; visual mesh filename=/home/gringo/ros2_ws/src/botzo/botzo_ros2_ws/botzo_descript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 scale=0.001 0.001 0.001
